Commit message: 0506

File: rg2_ws/src/rg2_description/urdf/rg2.urdf.xacro (robot description, xacro)
@@ -47,6 +47,6 @@
         <origin xyz="0.105 0.017 0.010" rpy="0 0 0"/>
         <axis xyz="0 0 1"/>
-        <limit velocity="3.14" effort="10.6" />
-        <limit lower="${gripper_lower_limit}" upper="${gripper_upper_limit}" />
+         <!-- 0505: TODO -->
+        <limit lower="${gripper_lower_limit}" upper="${gripper_upper_limit}" velocity="3.14" effort="10.6"/>
         <dynamics damping="0.1" friction="0.0" />
         <implicitSpringDamper>True</implicitSpringDamper>
@@ -80,5 +80,4 @@
         <axis xyz="0 0 1"/>
         <limit velocity="3.14" effort="10.6" lower="${-pi*0.5}" upper="${pi*0.5}" />
-        <!-- <limit velocity="3.14" effort="100" lower="-3" upper="3" /> -->
         <mimic joint="gripper_joint" multiplier="-1"/>
         <dynamics damping="0.1" friction="0.0" />
@@ -158,5 +157,5 @@
         <origin xyz="0.105 -0.017 0.010" rpy="0 0 0"/>
         <axis xyz="0 0 1"/>
-        <limit velocity="3.14" effort="10.6" lower="${-pi*0.5}" upper="${pi*0.5}" />
+        <limit lower="${gripper_lower_limit}" upper="${gripper_upper_limit}" effort="10.6" velocity="3.14" />
         <!-- <limit velocity="3.14" effort="100" lower="-3" upper="3" /> -->
         <mimic joint="gripper_joint" multiplier="-1"/>
